File: screenly-cm5-player/pcb/pcie.kicad_sch (KiCad schematic)
At the start: 17 parts, among them J4 SM3ZS067U410AMR1000, U4 LMR51450SDRRR

Commit message: WIP Schematics
Parts:
- added C26: 100nF, Screenly:C_0402, symbol Screenly:Capacitor 100nF 50V X7R 0402 (CL05B104KB54PNC)
- added R15: 10K, Screenly:R_0402, symbol Screenly:Resistor 10K 1% 0402 (RC0402FR-0710KL)
Connections:
- net GND: now also C26.1
- net PCIE_PG: now also C26.2, R15.2
- new net +3V3: R15.1

Commit message: Finished schematics design.
Parts:
- added TP13, TP14: TestPoint, Screenly:TestPoint_Pad_D2.0mm, symbol Screenly:Test Point Pad 2.0mm
- renumbered C17 to C19, C18 to C20, C19 to C21, C28 to C22, C21 to C23, C26 to C24, C22 to C25, C23 to C26, C24 to C27, C25 to C28, J4 to J5, R20 to R21, R19 to R22, R15 to R23, R12 to R24, R13 to R25, R16 to R26
Connections:
- net +3V3_PCIE: now also TP14.1
- net PCIE_PG: now also TP13.1
Other:
- moved on the sheet: C23
