File: screenly-cm5-player/pcb/user_interface.kicad_sch (KiCad schematic)
At the start: 16 parts, among them SW1 PTS645VM31-2, SW2 PTS645VM31-2

Commit message: New square shape
Added Raspberry Pi Antenna Kit
Parts:
- SW1, SW2: footprint Screenly:SW_Tactile_SPST_Angled_PTS645Vx31-2LFS -> Screenly:SW_Tactile_SPST_Angled_PTS645Vx58-2LFS; symbol Screenly:Tactile Switch 6x6mm 1.6N 3.15mm Right Angle THT (PTS645VM31-2 LFS) -> Screenly:Tactile Switch 6x6mm 1.6N 5.85mm Right Angle THT (PTS645VM58-2 LFS); MfrPartNum PTS645VM31-2 LFS -> PTS645VM58-2 LFS; PartNumber SRLY-SWC-000001 -> SRLY-SWC-000002; family PTS645V?31-2* -> PTS645V?58-2*; height 3.15mm -> 5.85mm
Changed lines of the file:
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@@
 	)
 	(symbol
-		(lib_id "Screenly:Tactile Switch 6x6mm 1.6N 3.15mm Right Angle THT (PTS645VM31-2 LFS)")
+		(lib_id "Screenly:Tactile Switch 6x6mm 1.6N 5.85mm Right Angle THT (PTS645VM58-2 LFS)")
 		(at 100.33 83.82 0)
 		(unit 1)
@@
 			)
 		)
-		(property "Footprint" "Screenly:SW_Tactile_SPST_Angled_PTS645Vx31-2LFS"
+		(property "Footprint" "Screenly:SW_Tactile_SPST_Angled_PTS645Vx58-2LFS"
 			(at 100.33 83.82 0)
 			(hide yes)
@@
 			)
 		)
-		(property "Description" "Tactile switch, SPST-NO, momentary, 6 x 6 mm, right angle (actuator parallel to the board), through hole, actuator 3.15 mm above the board, 160gf (1.6N) operating force, 50mA 12V DC, 100,000 operations, -40C to 85C. Pins 1 and 2 switch contacts, SH metal bracket legs (tie to GND for ESD)"
+		(property "Description" "Tactile switch, SPST-NO, momentary, 6 x 6 mm, right angle (actuator parallel to the board), through hole, actuator length L 5.85 mm from the front pin row (about 3.3 mm beyond the switch body), 160gf (1.6N) operating force, 50mA 12V DC, 100,000 operations, -40C to 85C. Pins 1 and 2 switch contacts, SH metal bracket legs (tie to GND for ESD)"
 			(at 100.33 83.82 0)
 			(hide yes)
@@
 			)
 		)
-		(property "PartNumber" "SRLY-SWC-000001"
+		(property "PartNumber" "SRLY-SWC-000002"
 			(at 100.33 83.82 0)
 			(hide yes)
@@
 			)
 		)
-		(property "MfrPartNum" "PTS645VM31-2 LFS"
+		(property "MfrPartNum" "PTS645VM58-2 LFS"
 			(at 100.33 83.82 0)
 			(hide yes)
@@
 			)
 		)
-		(property "family" "PTS645V?31-2*"
+		(property "family" "PTS645V?58-2*"
 			(at 100.33 83.82 0)
 			(hide yes)
@@
 			)
 		)
-		(property "height" "3.15mm"
+		(property "height" "5.85mm"
 			(at 100.33 83.82 0)
 			(hide yes)
@@
 	)
 	(symbol
-		(lib_id "Screenly:Tactile Switch 6x6mm 1.6N 3.15mm Right Angle THT (PTS645VM31-2 LFS)")
+		(lib_id "Screenly:Tactile Switch 6x6mm 1.6N 5.85mm Right Angle THT (PTS645VM58-2 LFS)")
 		(at 100.33 44.45 0)
 		(unit 1)
@@
 			)
 		)
-		(property "Footprint" "Screenly:SW_Tactile_SPST_Angled_PTS645Vx31-2LFS"
+		(property "Footprint" "Screenly:SW_Tactile_SPST_Angled_PTS645Vx58-2LFS"
 			(at 100.33 44.45 0)
 			(hide yes)
@@
 			)
 		)
-		(property "Description" "Tactile switch, SPST-NO, momentary, 6 x 6 mm, right angle (actuator parallel to the board), through hole, actuator 3.15 mm above the board, 160gf (1.6N) operating force, 50mA 12V DC, 100,000 operations, -40C to 85C. Pins 1 and 2 switch contacts, SH metal bracket legs (tie to GND for ESD)"
+		(property "Description" "Tactile switch, SPST-NO, momentary, 6 x 6 mm, right angle (actuator parallel to the board), through hole, actuator length L 5.85 mm from the front pin row (about 3.3 mm beyond the switch body), 160gf (1.6N) operating force, 50mA 12V DC, 100,000 operations, -40C to 85C. Pins 1 and 2 switch contacts, SH metal bracket legs (tie to GND for ESD)"
 			(at 100.33 44.45 0)
 			(hide yes)
@@
 			)
 		)
-		(property "PartNumber" "SRLY-SWC-000001"
+		(property "PartNumber" "SRLY-SWC-000002"
 			(at 100.33 44.45 0)
 			(hide yes)
@@
 			)
 		)
-		(property "MfrPartNum" "PTS645VM31-2 LFS"
+		(property "MfrPartNum" "PTS645VM58-2 LFS"
 			(at 100.33 44.45 0)
 			(hide yes)
@@
 			)
 		)
-		(property "family" "PTS645V?31-2*"
+		(property "family" "PTS645V?58-2*"
 			(at 100.33 44.45 0)
 			(hide yes)
@@
 			)
 		)
-		(property "height" "3.15mm"
+		(property "height" "5.85mm"
 			(at 100.33 44.45 0)
 			(hide yes)
