File: screenly-cm5-player/pcb/compute_module.kicad_sch (KiCad schematic)
At the start: 4 parts, among them J1 CR2032 Holder, U1 CM5104064

Commit message: Finished schematics design.
Parts:
- removed J1: CR2032 Holder, Screenly:BatteryHolder_MYOUNG_BS-02_CR2032, symbol Screenly:Battery Holder CR2032 THT (BS-02-A1AJ010)
- added J1: CR2032 Retainer, Screenly:BatteryHolder_MYOUNG_MY-2032-08_CR2032, symbol Screenly:Battery Holder CR2032 SMD Retainer (MY-2032-08)
- added J2: BM03B-SRSS-TB, Screenly:JST_SH_BM03B-SRSS-TB_1x03-1MP_P1.00mm_Vertical, symbol Screenly:JST SH Header 3P 1.0mm Vertical SMD (BM03B-SRSS-TB)
- added R2, R5: 33R, Screenly:R_0402, symbol Screenly:Resistor 33R 5% 0402 (RC0402JR-0733RL)
- added R3, R4: 120, Screenly:R_0402, symbol Screenly:Resistor 120R 5% 0402 (0402WGJ0121TCE)
- added TP1, TP2, TP3, TP4, TP5: TestPoint, Screenly:TestPoint_Pad_D2.0mm, symbol Screenly:Test Point Pad 2.0mm
- renumbered R14 to R1, R33 to R6
Connections:
- net +1V8: now also TP2.1
- net +3V3: now also TP1.1
- net +BATT: now also J1.1 (+)
- net GND: now also J1.2 (-), J2.2 (Pin_2), J2.MP, TP5.1
- net PCIE_PG: now also U1.24 (GPIO26)
- net USB_PG: now also U1.50 (GPIO17)
- net ~{HDMI0_PWR_FAULT}: now also U1.34 (GPIO5)
- net ~{HDMI1_PWR_FAULT}: now also U1.30 (GPIO6)
- net ~{USB3_0_PWR_FAULT}: now also U1.46 (GPIO22)
- net ~{USB3_1_PWR_FAULT}: now also U1.47 (GPIO23)
- net EE_SCL: now reaches U1.35 (ID_SC)
- net EE_SDA: now reaches U1.36 (ID_SD)
- net TPM.~{CS}: now reaches U1.37 (GPIO7)
- net TPM.CLK: now reaches U1.38 (GPIO11)
- net TPM.MISO: now reaches U1.40 (GPIO9)
- net ~{TPM_PIRQ}: now reaches U1.41 (GPIO25)
- net TPM.MOSI: now reaches U1.44 (GPIO10)
- net ~{TPM_RST}: now reaches U1.45 (GPIO24)
- net ~{USB2_PWR_FAULT}: now reaches U1.48 (GPIO27)
- net A_SCLK: now reaches U1.49 (GPIO18)
- net A_SCLK: now also R5.1
- net DBG_RX: now reaches U1.51 (GPIO15)
- net DBG_RX: now also R3.1
- net ~{FACTORY_RST_BTN}: now reaches U1.54 (GPIO4)
- net DBG_TX: now reaches U1.55 (GPIO14)
- net DBG_TX: now also R4.1
- net CAM_GPIO1: no longer names the net of U1.100 (CAM_GPIO1)
- net CC1: no longer names the net of U1.94 (CC1)
- net CC2: no longer names the net of U1.96 (CC2)
- net DPHY0_P.C_N: no longer names the net of U1.127 (MIPI0_C_N)
- net DPHY0_P.C_P: no longer names the net of U1.129 (MIPI0_C_P)
- net DPHY0_P.D0_N: no longer names the net of U1.115 (MIPI0_D0_N)
- net DPHY0_P.D0_P: no longer names the net of U1.117 (MIPI0_D0_P)
- net DPHY0_P.D1_N: no longer names the net of U1.121 (MIPI0_D1_N)
- net DPHY0_P.D1_P: no longer names the net of U1.123 (MIPI0_D1_P)
- net DPHY0_P.D2_N: no longer names the net of U1.133 (MIPI0_D2_N)
- net DPHY0_P.D2_P: no longer names the net of U1.135 (MIPI0_D2_P)
- net DPHY0_P.D3_N: no longer names the net of U1.139 (MIPI0_D3_N)
- net DPHY0_P.D3_P: no longer names the net of U1.141 (MIPI0_D3_P)
- net DPHY1_P.C_N: no longer names the net of U1.187 (MIPI1_C_N)
- net DPHY1_P.C_P: no longer names the net of U1.189 (MIPI1_C_P)
- net DPHY1_P.D0_N: no longer names the net of U1.175 (MIPI1_D0_N)
- net DPHY1_P.D0_P: no longer names the net of U1.177 (MIPI1_D0_P)
- net DPHY1_P.D1_N: no longer names the net of U1.181 (MIPI1_D1_N)
- net DPHY1_P.D1_P: no longer names the net of U1.183 (MIPI1_D1_P)
- net DPHY1_P.D2_N: no longer names the net of U1.193 (MIPI1_D2_N)
- net DPHY1_P.D2_P: no longer names the net of U1.195 (MIPI1_D2_P)
- net DPHY1_P.D3_N: no longer names the net of U1.194 (MIPI1_D3_N)
- net DPHY1_P.D3_P: no longer names the net of U1.196 (MIPI1_D3_P)
- net GLOBAL_EN: no longer names the net of U1.99 (PMIC_ENABLE)
- net MISO_GPIO19 renamed A_WS
- net A_WS: now also R2.2
- net MOSI_GPIO20: no longer names the net of U1.27 (GPIO20)
- net SCLK_GPIO21 renamed Audio.SDO0
- net SD_CARD.D4: no longer names the net of U1.68 (SD_DAT4)
- net SD_CARD.D5: no longer names the net of U1.64 (SD_DAT5)
- net SD_CARD.D6: no longer names the net of U1.72 (SD_DAT6)
- net SD_CARD.D7: no longer names the net of U1.70 (SD_DAT7)
- net USBOTG_ID: no longer names the net of U1.101 (USB_OTG_ID)
- new net Audio.SCLK: R5.2
- new net Audio.WS: R2.1
- new net DBG_RX_F: J2.1 (Pin_1), R3.2, TP4.1
- new net DBG_TX_F: J2.3 (Pin_3), R4.2, TP3.1
- no-connect marks 48 -> 45
Other:
- note added: "Keep this resistor close to CM5 connector"

Commit message: New square shape
Added Raspberry Pi Antenna Kit
Parts:
- added MK1: Antenna Kit Outline, Screenly:RaspberryPi_Antenna_Kit_Outline_SideView, symbol Screenly:Mechanical Outline Raspberry Pi Antenna Kit
Changed lines of the file:
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@@
+	)
+	(symbol
+		(lib_id "Screenly:Mechanical Outline Raspberry Pi Antenna Kit")
+		(at 142.24 181.61 0)
+		(unit 1)
+		(body_style 1)
+		(exclude_from_sim yes)
+		(in_bom no)
+		(on_board yes)
+		(in_pos_files no)
+		(dnp no)
+		(fields_autoplaced yes)
+		(property "Reference" "MK1"
+			(at 144.78 179.5779 0)
+			(show_name no)
+			(do_not_autoplace no)
+			(effects
+				(font
+					(size 1.27 1.27)
+				)
+				(justify left)
+			)
+		)
+		(property "Value" "Antenna Kit Outline"
+			(at 144.78 182.1179 0)
+			(show_name no)
+			(do_not_autoplace no)
+			(effects
+				(font
+					(size 1.27 1.27)
+				)
+				(justify left)
+			)
+		)
+		(property "Footprint" "Screenly:RaspberryPi_Antenna_Kit_Outline_SideView"
+			(at 142.24 181.61 0)
+			(hide yes)
+			(show_name no)
+			(do_not_autoplace no)
+			(effects
+				(font
+					(size 1.27 1.27)
+				)
+			)
+		)
+		(property "Datasheet" "https://datasheets.raspberrypi.com/cm4/cm4-antenna-kit-product-brief.pdf"
+			(at 142.24 181.61 0)
+			(hide yes)
+			(show_name no)
+			(do_not_autoplace no)
+			(effects
+				(font
+					(size 1.27 1.27)
+				)
+			)
+		)
+		(property "Description" "Mechanical outline of the Raspberry Pi Antenna Kit (folded antenna on the SMA bulkhead), side view on Dwgs.User, for board-edge and enclosure placement. Not a part: excluded from BOM and position files. The antenna kit itself is a separate off-board ANT item"
+			(at 142.24 181.61 0)
+			(hide yes)
+			(show_name no)
+			(do_not_autoplace no)
+			(effects
+				(font
+					(size 1.27 1.27)
+				)
+			)
+		)
+		(instances
+			(project "screenly-cm5-player"
+				(path "/e8a2875a-18ea-4799-b56d-ecb6ae09ef8e/3fbfb189-ea05-4055-8850-fa2523ec0120"
+					(reference "MK1")
+					(unit 1)
+				)
+			)
+		)
 	)
 	(symbol

Commit message: Rough placements
Parts:
- added J14, J15: DF40HC(3.0)-100DS-0.4V, Screenly:Hirose_DF40HC-3.0-100DS-0.4V_2x50_P0.4mm_Vertical_NoCopper, symbol Screenly:Board to Board Receptacle 100P 0.4mm 3.0mm Stack SMD (DF40HC(3.0)-100D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
- U1: now left out of the parts list
Other:
- note added: "J14 and J15 are the actual connectors for the CM5 module to be populated at the assembly. But they are only for mechanical reference."
- moved on the sheet: J1, J2, MK1, R3, R4, TP3, TP4, TP5
