File: screenly-cm5-player/pcb/ethernet.kicad_sch (KiCad schematic)
At the start: 6 parts, among them J3 HB-W01G0520DQW-R

Commit message: WIP Schematics
Parts:
- removed D3, D4: TPD4EUSB30DQAR, Screenly:TI_USON-10_2.5x1.0mm_P0.5mm, symbol Screenly:ESD Diode 4ch 5.5V USON-10 (TPD4EUSB30DQAR)
- added D3, D4: TPD4E05U06DQAR, Screenly:TI_USON-10_2.5x1.0mm_P0.5mm, symbol Screenly:ESD Diode 4ch 5.5V USON-10 (TPD4E05U06DQAR)
Connections:
- net ETH.TRD0_N: now also D3.2 (D1-), D3.9
- net ETH.TRD0_P: now also D3.1 (D1+), D3.10
- net ETH.TRD1_N: now also D3.5 (D2-), D3.6
- net ETH.TRD1_P: now also D3.4 (D2+), D3.7
- net ETH.TRD2_N: now also D4.2 (D1-), D4.9
- net ETH.TRD2_P: now also D4.1 (D1+), D4.10
- net ETH.TRD3_N: now also D4.5 (D2-), D4.6
- net ETH.TRD3_P: now also D4.4 (D2+), D4.7
- net GND: now also D3.3 (GND), D3.8 (GND), D4.3 (GND), D4.8 (GND)

Commit message: Finished schematics design.
Parts:
- renumbered C27 to C18, J3 to J4, R18 to R19, R17 to R20
Connections:
- net ETH.TRD1_N: no longer D3.6
- net ETH.TRD1_P: no longer D3.7
- net ETH.TRD3_N: no longer D4.6
- net ETH.TRD3_P: no longer D4.7
Changed lines of the file:
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@@
 		(dnp no)
 		(fields_autoplaced yes)
-		(property "Reference" "C27"
+		(property "Reference" "C18"
 			(at 186.69 96.5199 0)
 			(show_name no)
@@
 			(project "screenly-cm5-player"
 				(path "/e8a2875a-18ea-4799-b56d-ecb6ae09ef8e/c23b474a-a5df-4d03-b71c-bc870a6cf46c"
-					(reference "C27")
+					(reference "C18")
 					(unit 1)
 				)
@@
 		(dnp no)
 		(fields_autoplaced yes)
-		(property "Reference" "J3"
+		(property "Reference" "J4"
 			(at 203.2 66.04 0)
 			(show_name no)
@@
 			(project "screenly-cm5-player"
 				(path "/e8a2875a-18ea-4799-b56d-ecb6ae09ef8e/c23b474a-a5df-4d03-b71c-bc870a6cf46c"
-					(reference "J3")
+					(reference "J4")
 					(unit 1)
 				)
@@
 		(dnp no)
 		(fields_autoplaced yes)
-		(property "Reference" "#PWR052"
+		(property "Reference" "#PWR046"
 			(at 203.2 105.41 0)
 			(hide yes)
@@
 			(project "screenly-cm5-player"
 				(path "/e8a2875a-18ea-4799-b56d-ecb6ae09ef8e/c23b474a-a5df-4d03-b71c-bc870a6cf46c"
-					(reference "#PWR052")
+					(reference "#PWR046")
 					(unit 1)
 				)
@@
 		(dnp no)
 		(fields_autoplaced yes)
-		(property "Reference" "R18"
+		(property "Reference" "R19"
 			(at 224.79 86.3599 0)
 			(show_name no)
@@
 			(project "screenly-cm5-player"
 				(path "/e8a2875a-18ea-4799-b56d-ecb6ae09ef8e/c23b474a-a5df-4d03-b71c-bc870a6cf46c"
-					(reference "R18")
+					(reference "R19")
 					(unit 1)
 				)
@@
 		(in_pos_files yes)
 		(dnp no)
-		(property "Reference" "#PWR047"
+		(property "Reference" "#PWR048"
 			(at 222.25 71.12 0)
 			(hide yes)
@@
 			(project "screenly-cm5-player"
 				(path "/e8a2875a-18ea-4799-b56d-ecb6ae09ef8e/c23b474a-a5df-4d03-b71c-bc870a6cf46c"
-					(reference "#PWR047")
+					(reference "#PWR048")
 					(unit 1)
 				)
@@
 		(dnp no)
 		(fields_autoplaced yes)
-		(property "Reference" "#PWR049"
+		(property "Reference" "#PWR044"
 			(at 139.7 135.89 0)
 			(hide yes)
@@
 			(project "screenly-cm5-player"
 				(path "/e8a2875a-18ea-4799-b56d-ecb6ae09ef8e/c23b474a-a5df-4d03-b71c-bc870a6cf46c"
-					(reference "#PWR049")
+					(reference "#PWR044")
 					(unit 1)
 				)
@@
 		(dnp no)
 		(fields_autoplaced yes)
-		(property "Reference" "#PWR051"
+		(property "Reference" "#PWR047"
 			(at 218.44 90.17 0)
 			(hide yes)
@@
 			(project "screenly-cm5-player"
 				(path "/e8a2875a-18ea-4799-b56d-ecb6ae09ef8e/c23b474a-a5df-4d03-b71c-bc870a6cf46c"
-					(reference "#PWR051")
+					(reference "#PWR047")
 					(unit 1)
 				)
@@
 		(dnp no)
 		(fields_autoplaced yes)
-		(property "Reference" "#PWR048"
+		(property "Reference" "#PWR043"
 			(at 96.52 135.89 0)
 			(hide yes)
@@
 			(project "screenly-cm5-player"
 				(path "/e8a2875a-18ea-4799-b56d-ecb6ae09ef8e/c23b474a-a5df-4d03-b71c-bc870a6cf46c"
-					(reference "#PWR048")
+					(reference "#PWR043")
 					(unit 1)
 				)
@@
 		(dnp no)
 		(fields_autoplaced yes)
-		(property "Reference" "#PWR050"
+		(property "Reference" "#PWR045"
 			(at 182.88 107.95 0)
 			(hide yes)
@@
 			(project "screenly-cm5-player"
 				(path "/e8a2875a-18ea-4799-b56d-ecb6ae09ef8e/c23b474a-a5df-4d03-b71c-bc870a6cf46c"
-					(reference "#PWR050")
+					(reference "#PWR045")
 					(unit 1)
 				)
@@
 		(dnp no)
 		(fields_autoplaced yes)
-		(property "Reference" "R17"
+		(property "Reference" "R20"
 			(at 233.68 86.3599 0)
 			(show_name no)
@@
 			(project "screenly-cm5-player"
 				(path "/e8a2875a-18ea-4799-b56d-ecb6ae09ef8e/c23b474a-a5df-4d03-b71c-bc870a6cf46c"
-					(reference "R17")
+					(reference "R20")
 					(unit 1)
 				)

Commit message: Rough placements
Connections:
- net ETH.TRD1_N: now also D3.4 (D2+), D3.7; no longer D3.5 (D2-)
- net ETH.TRD1_P: now also D3.5 (D2-), D3.6; no longer D3.4 (D2+)
- net ETH.TRD3_N: now also D4.4 (D2+), D4.7; no longer D4.5 (D2-)
- net ETH.TRD3_P: now also D4.5 (D2-), D4.6; no longer D4.4 (D2+)
Changed lines of the file:
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@@
-	)
-	(junction
-		(at 114.3 81.28)
-		(diameter 0)
-		(color 0 0 0 0)
 	)
 	(junction
@@
 	)
 	(junction
-		(at 157.48 91.44)
-		(diameter 0)
-		(color 0 0 0 0)
-	)
-	(junction
-		(at 111.76 78.74)
+		(at 111.76 81.28)
+		(diameter 0)
+		(color 0 0 0 0)
+	)
+	(junction
+		(at 114.3 78.74)
 		(diameter 0)
 		(color 0 0 0 0)
@@
 	)
 	(junction
-		(at 154.94 88.9)
+		(at 154.94 91.44)
+		(diameter 0)
+		(color 0 0 0 0)
+	)
+	(junction
+		(at 157.48 88.9)
 		(diameter 0)
 		(color 0 0 0 0)
@@
 	(wire
 		(pts
+			(xy 153.67 114.3) (xy 152.4 114.3)
+		)
+		(stroke
+			(width 0)
+			(type default)
+		)
+	)
+	(wire
+		(pts
 			(xy 68.58 86.36) (xy 121.92 86.36)
 		)
@@
 	(wire
 		(pts
-			(xy 152.4 119.38) (xy 157.48 119.38)
+			(xy 114.3 78.74) (xy 187.96 78.74)
+		)
+		(stroke
+			(width 0)
+			(type default)
+		)
+	)
+	(wire
+		(pts
+			(xy 156.21 116.84) (xy 157.48 116.84)
+		)
+		(stroke
+			(width 0)
+			(type default)
+		)
+	)
+	(wire
+		(pts
+			(xy 111.76 81.28) (xy 111.76 114.3)
 		)
 		(stroke
@@
 	(wire
 		(pts
-			(xy 111.76 78.74) (xy 187.96 78.74)
-		)
-		(stroke
-			(width 0)
-			(type default)
-		)
-	)
-	(wire
-		(pts
-			(xy 154.94 88.9) (xy 187.96 88.9)
+			(xy 68.58 78.74) (xy 114.3 78.74)
+		)
+		(stroke
+			(width 0)
+			(type default)
+		)
+	)
+	(wire
+		(pts
+			(xy 68.58 88.9) (xy 157.48 88.9)
 		)
 		(stroke
@@
 	(wire
 		(pts
+			(xy 153.67 116.84) (xy 153.67 114.3)
+		)
+		(stroke
+			(width 0)
+			(type default)
+		)
+	)
+	(wire
+		(pts
 			(xy 222.25 91.44) (xy 222.25 95.25)
 		)
@@
 	(wire
 		(pts
-			(xy 157.48 119.38) (xy 157.48 91.44)
-		)
-		(stroke
-			(width 0)
-			(type default)
-		)
-	)
-	(wire
-		(pts
-			(xy 154.94 114.3) (xy 154.94 88.9)
-		)
-		(stroke
-			(width 0)
-			(type default)
-		)
-	)
-	(wire
-		(pts
-			(xy 152.4 114.3) (xy 154.94 114.3)
+			(xy 157.48 116.84) (xy 157.48 88.9)
+		)
+		(stroke
+			(width 0)
+			(type default)
+		)
+	)
+	(wire
+		(pts
+			(xy 154.94 116.84) (xy 154.94 91.44)
+		)
+		(stroke
+			(width 0)
+			(type default)
+		)
+	)
+	(wire
+		(pts
+			(xy 153.67 116.84) (xy 154.94 116.84)
 		)
 		(stroke
@@
 	(wire
 		(pts
+			(xy 156.21 116.84) (xy 156.21 119.38)
+		)
+		(stroke
+			(width 0)
+			(type default)
+		)
+	)
+	(wire
+		(pts
+			(xy 154.94 91.44) (xy 187.96 91.44)
+		)
+		(stroke
+			(width 0)
+			(type default)
+		)
+	)
+	(wire
+		(pts
 			(xy 109.22 114.3) (xy 111.76 114.3)
 		)
@@
 	(wire
 		(pts
-			(xy 68.58 78.74) (xy 111.76 78.74)
+			(xy 109.22 119.38) (xy 114.3 119.38)
 		)
 		(stroke
@@
 	(wire
 		(pts
-			(xy 114.3 81.28) (xy 187.96 81.28)
-		)
-		(stroke
-			(width 0)
-			(type default)
-		)
-	)
-	(wire
-		(pts
-			(xy 68.58 88.9) (xy 154.94 88.9)
-		)
-		(stroke
-			(width 0)
-			(type default)
-		)
-	)
-	(wire
-		(pts
-			(xy 68.58 91.44) (xy 157.48 91.44)
+			(xy 111.76 81.28) (xy 187.96 81.28)
+		)
+		(stroke
+			(width 0)
+			(type default)
+		)
+	)
+	(wire
+		(pts
+			(xy 157.48 88.9) (xy 187.96 88.9)
+		)
+		(stroke
+			(width 0)
+			(type default)
+		)
+	)
+	(wire
+		(pts
+			(xy 68.58 91.44) (xy 154.94 91.44)
 		)
 		(stroke
@@
 		)
 	)
-	(wire
-		(pts
-			(xy 109.22 119.38) (xy 114.3 119.38)
-		)
-		(stroke
-			(width 0)
-			(type default)
-		)
-	)
 	(bus
 		(pts
@@
 	(wire
 		(pts
-			(xy 111.76 114.3) (xy 111.76 78.74)
-		)
-		(stroke
-			(width 0)
-			(type default)
-		)
-	)
-	(wire
-		(pts
-			(xy 114.3 119.38) (xy 114.3 81.28)
+			(xy 114.3 119.38) (xy 114.3 78.74)
 		)
 		(stroke
@@
 	(wire
 		(pts
-			(xy 68.58 81.28) (xy 114.3 81.28)
+			(xy 156.21 119.38) (xy 152.4 119.38)
+		)
+		(stroke
+			(width 0)
+			(type default)
+		)
+	)
+	(wire
+		(pts
+			(xy 68.58 81.28) (xy 111.76 81.28)
 		)
 		(stroke
@@
 		)
 		(stroke
-			(width 0)
-			(type default)
-		)
-	)
-	(wire
-		(pts
-			(xy 157.48 91.44) (xy 187.96 91.44)
-		)
-		(stroke
