File: screenly-cm5-player/pcb/hdmi.kicad_sch (KiCad schematic)
At the start: 22 parts, among them J5 2086581001, J6 2086581001, U5 AP22652W6-7, U6 AP22652W6-7

Commit message: Finished schematics design.
Parts:
- removed U5, U6: AP22652W6-7, Screenly:SOT-23-6, symbol Screenly:Power Switch 3-5.5V 2.1A SOT-23-6 (AP22652W6-7)
- added U5, U6: AP22653W6-7, Screenly:SOT-23-6, symbol Screenly:Power Switch 3-5.5V 2.1A SOT-23-6 (AP22653W6-7)
- renumbered C30 to C29, C32 to C30, C34 to C31, C35 to C32, C31 to C33, C33 to C34, D8 to D6, D6 to D7, D9 to D8, D7 to D9, J5 to J6, J6 to J7, R22 to R27, R23 to R28, R24 to R29, R25 to R30, R21 to R31, R27 to R32
Connections:
- net +5V: now also U5.1 (IN), U5.3 (EN), U6.1 (IN), U6.3 (EN)
- net GND: now also U5.2 (GND), U6.2 (GND)
- net HDMI0.CEC: no longer D9.7
- net HDMI0.CK_N: no longer D7.6
- net HDMI0.CK_P: no longer D7.7
- net HDMI0.D1_N: no longer D5.6
- net HDMI0.D1_P: no longer D5.7
- net HDMI0.HOTPLUG: no longer D9.6
- net HDMI1.CEC: no longer D10.7
- net HDMI1.CK_N: no longer D8.6
- net HDMI1.CK_P: no longer D8.7
- net HDMI1.D1_N: no longer D6.6
- net HDMI1.D1_P: no longer D6.7
- net HDMI1.HOTPLUG: no longer D10.6
- net at R30.1: now also U6.5 (ILIM)
- net at C29.1, C31.1, J6.18 (+5V): now also U5.6 (OUT)
- net at C30.1, C32.1, J7.18 (+5V): now also U6.6 (OUT)
- net at R28.1: now also U6.4 (~{FAULT})
- net at R29.1: now also U5.5 (ILIM)
- net at R27.1: now also U5.4 (~{FAULT})

Commit message: Rough placements
Connections:
- net HDMI0.CEC: now also D9.7
- net HDMI0.CK_N: now also D7.6
- net HDMI0.CK_P: now also D7.7
- net HDMI0.D1_N: now also D5.6
- net HDMI0.D1_P: now also D5.7
- net HDMI0.HOTPLUG: now also D9.6
- net HDMI1.CEC: now also D10.7
- net HDMI1.CK_N: now also D8.6
- net HDMI1.CK_P: now also D8.7
- net HDMI1.D1_N: now also D6.6
- net HDMI1.D1_P: now also D6.7
- net HDMI1.HOTPLUG: now also D10.6
