File: screenly-cm5-player/pcb/power.kicad_sch (KiCad schematic)
At the start: 49 parts, among them J2 DC Jack 5.5x2.1mm, Q1 AOD4185, U2 LMR51450SDRRR, U3 LMR51450SDRRR, U4 LMR51450SDRRR

Commit message: Ethernet and PCIe sections are done.
Modified power section and moved PCIe specific circuit into its own
section.
Parts:
- removed C17, C18: 10uF, Screenly:C_1210, symbol Screenly:Capacitor 10uF 50V X7R 1210 (CL32B106KBJNNNE)
- removed C19, C21: 100nF, Screenly:C_0402, symbol Screenly:Capacitor 100nF 50V X7R 0402 (CL05B104KB54PNC)
- removed C22: 33pF, Screenly:C_0402, symbol Screenly:Capacitor 33pF 50V C0G 0402 (CL05C330JB5NNNC)
- removed C23, C24, C25: 47uF, Screenly:C_1210, symbol Screenly:Capacitor 47uF 10V X7R 1210 (GRM32ER71A476KE15L)
- removed L3: 4.7uH, Screenly:L_Coilank_AAPS1050, symbol Screenly:Inductor 4.7uH 15A 10x11.5mm (AAPS1050M4R7A)
- removed R12: 100K, Screenly:R_0402, symbol Screenly:Resistor 100K 1% 0402 (0402WGF1003TCE)
- removed R13: 31.6K, Screenly:R_0402, symbol Screenly:Resistor 31.6K 1% 0402 (0402WGF3162TCE)
- removed R16: 1K, Screenly:R_0402, symbol Screenly:Resistor 1K 5% 0402 (0402WGJ0102TCE)
- removed R4, R9: 19.1K, Screenly:R_0402, symbol Screenly:Resistor 19.1K 1% 0402 (0402WGF1912TCE)
- removed U4: LMR51450SDRRR, Screenly:TI_WSON-12-1EP_3x3mm_P0.5mm_EP1.3x2.5mm, symbol Screenly:Buck Converter 4-36V 5A WSON-12 (LMR51450SDRRR)
- added R4, R9: 19.1K, Screenly:R_0402, symbol Screenly:Resistor 19.1K 1% 0402 (GR0402F19K1TAG00)
Connections:
- net GND: now also R4.2, R9.2
- net at C12.1, R8.2, U3.7 (FB): now also R9.1
- net at C5.1, R3.2, U2.7 (FB): now also R4.1
- no-connect marks 4 -> 3
Other:
- moved on the sheet: C1, C10, C11, C12, C13, C14, C15, C16, C2, C3, C4, C5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

Commit message: WIP Schematics
Parts:
- removed C16: 100uF, Screenly:CP_Elec_6.3x7.7, symbol Screenly:Capacitor 100uF 35V Electrolytic 6.3x7.7mm (EEE-FK1V101XP)
- added C16: 220uF, Screenly:CP_Radial_D6.3mm_P2.50mm, symbol Screenly:Capacitor 220uF 35V Polymer Radial 6.3x11mm (PPH1V221M061100N)
- added C29: 120uF, Screenly:CP_Elec_6.3x5.9, symbol Screenly:Capacitor 120uF 10V Polymer 6.3x5.9mm (OVZ121M1ATR-0606)
Connections:
- net +12V: now also C16.1
- net +5V_USB: now also C29.1
- net GND: now also C16.2, C29.2
Other:
- note added: "// TODO: Connect reset button to the EN input of U2"

Commit message: Finished schematics design.
Parts:
- added R12: 10K, Screenly:R_0402, symbol Screenly:Resistor 10K 1% 0402 (RC0402FR-0710KL)
- added TP10, TP11, TP12, TP6, TP7, TP8, TP9: TestPoint, Screenly:TestPoint_Pad_D2.0mm, symbol Screenly:Test Point Pad 2.0mm
- renumbered C16 to C1, C11 to C10, C5 to C11, C6 to C13, C13 to C14, C7 to C15, C14 to C16, C29 to C17, C1 to C2, C8 to C3, C2 to C4, C9 to C5, C3 to C6, C10 to C7, C15 to C8, C4 to C9, J2 to J3, R1 to R10, R3 to R13, R4 to R14, R8 to R15, R9 to R16, R5 to R17, R10 to R18, R6 to R8, R2 to R9
Connections:
- net +12V: now also TP8.1
- net +5V: now also TP11.1
- net +5V_USB: now also TP12.1
- net GND: now also TP6.1
- net MAIN_5V_PG: now also TP9.1
- net USB_PG: now also R12.2, TP10.1
- net at D1.2 (A2), J3.1, Q1.2 (D): now also TP7.1
- new net +3V3: R12.1
Other:
- note removed: "// TODO: Connect reset button to the EN input of U2"
- moved on the sheet: C1, C10, C9

Commit message: Rough placements
Connections:
- net GND: now also D1.2 (A2); no longer D1.1 (A1)
- net at J3.1, Q1.2 (D), TP7.1: now also D1.1 (A1); no longer D1.2 (A2)
Other:
- moved on the sheet: D1
Changed lines of the file:
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@@
 	(symbol
 		(lib_id "Screenly:TVS Diode Bidirectional 18V 600W SMB (SMBJ18CA)")
-		(at 50.8 55.88 90)
+		(at 50.8 55.88 270)
 		(unit 1)
 		(body_style 1)
@@
 					(size 1.27 1.27)
 				)
-				(justify right)
+				(justify left)
 			)
 		)
@@
 					(size 1.27 1.27)
 				)
-				(justify right)
+				(justify left)
 			)
 		)
