File: screenly-cm5-player/pcb/screenly-cm5-player.kicad_pcb (KiCad board)
At the start: 2 copper layers, 120 x 90 mm, 65 parts, among them J1 CR2032 Holder, J2 DC Jack 5.5x2.1mm, J3 HB-W01G0520DQW-R, J4 SM3ZS067U410AMR1000, Q1 AOD4185, U1 CM5104064, U2 LMR51450SDRRR, U3 LMR51450SDRRR, U4 LMR51450SDRRR

Commit message: WIP Schematics
Parts:
- added C16: 220uF, Screenly:CP_Radial_D6.3mm_P2.50mm, F.Cu at (245.8, 135.9)
- added C26: 100nF, Screenly:C_0402, F.Cu at (244.5, 148.9)
- added C29: 120uF, Screenly:CP_Elec_6.3x5.9, F.Cu at (248.2, 127.9)
- added C30: 100nF, Screenly:C_0402, F.Cu at (236.4, 125.0)
- added C31: 100nF, Screenly:C_0402, F.Cu at (236.4, 126.9)
- added C32: 100nF, Screenly:C_0402, F.Cu at (236.4, 128.8)
- added C33: 100nF, Screenly:C_0402, F.Cu at (236.4, 130.7)
- added C34: 10uF, Screenly:C_1210, F.Cu at (237.6, 144.5)
- added C35: 10uF, Screenly:C_1210, F.Cu at (237.6, 148.6)
- added C36: 100nF, Screenly:C_0402, F.Cu at (180.1, 146.5)
- added C37: 10uF, Screenly:C_1210, F.Cu at (165.3, 161.9)
- added C38: 100nF, Screenly:C_0402, F.Cu at (180.1, 148.4)
- added D10: TPD4E05U06DQAR, Screenly:TI_USON-10_2.5x1.0mm_P0.5mm, F.Cu at (232.8, 154.5)
- added D3: TPD4E05U06DQAR, Screenly:TI_USON-10_2.5x1.0mm_P0.5mm, F.Cu at (244.4, 143.9)
- added D4: TPD4E05U06DQAR, Screenly:TI_USON-10_2.5x1.0mm_P0.5mm, F.Cu at (247.3, 143.9)
- added D5: TPD4E05U06DQAR, Screenly:TI_USON-10_2.5x1.0mm_P0.5mm, F.Cu at (218.4, 154.5)
- added D6: TPD4E05U06DQAR, Screenly:TI_USON-10_2.5x1.0mm_P0.5mm, F.Cu at (221.3, 154.5)
- added D7: TPD4E05U06DQAR, Screenly:TI_USON-10_2.5x1.0mm_P0.5mm, F.Cu at (224.2, 154.5)
- added D8: TPD4E05U06DQAR, Screenly:TI_USON-10_2.5x1.0mm_P0.5mm, F.Cu at (227.0, 154.5)
- added D9: TPD4E05U06DQAR, Screenly:TI_USON-10_2.5x1.0mm_P0.5mm, F.Cu at (229.9, 154.5)
- added J5: 2086581001, Screenly:HDMI_A_Molex_208658-1001_Horizontal, F.Cu at (133.2, 125.5)
- added J6: 2086581001, Screenly:HDMI_A_Molex_208658-1001_Horizontal, F.Cu at (151.2, 125.5)
- added J7: 10.0 QHHTZB6.3, Screenly:USB_A_SHOUHAN_QHHTZB6.3_Horizontal, F.Cu at (167.9, 134.0)
- added R14: 0, Screenly:SolderBridge_0402, F.Cu at (244.5, 154.8)
- added R15: 10K, Screenly:R_0402, F.Cu at (244.5, 150.8)
- added R21: 10K, Screenly:R_0402, F.Cu at (236.4, 132.6)
- added R22: 120, Screenly:R_0402, F.Cu at (239.4, 125.0)
- added R23: 120, Screenly:R_0402, F.Cu at (239.4, 126.9)
- added R24: 100K, Screenly:R_0402, F.Cu at (239.4, 128.8)
- added R25: 100K, Screenly:R_0402, F.Cu at (239.4, 130.7)
- added R26: 120, Screenly:R_0402, F.Cu at (180.1, 150.3)
- added R27: 10K, Screenly:R_0402, F.Cu at (239.4, 132.6)
- added R28: 100K, Screenly:R_0402, F.Cu at (180.1, 152.2)
- added R29: 10K, Screenly:R_0402, F.Cu at (180.1, 154.1)
- added U5: AP22652W6-7, Screenly:SOT-23-6, F.Cu at (237.3, 135.8)
- added U6: AP22652W6-7, Screenly:SOT-23-6, F.Cu at (237.3, 140.3)
- added U7: AP22652W6-7, Screenly:SOT-23-6, F.Cu at (170.5, 162.1)
Connections:
- R17 pad 2: /Compute Module/~{CM5_LED_ACT} -> /Compute Module/~{ETH_LED_ACT}
- R18 pad 2: /Compute Module/~{CM5_LED_PWR} -> /Compute Module/~{ETH_LED_SPD}
- U1 pad 20: /Compute Module/~{EEPROM_WP} -> Net-(U1A-EEPROM_nWP)
- U1 pad 35: /Compute Module/ID_SC -> unconnected-(U1A-ID_SC-Pad35)
- U1 pad 36: /Compute Module/ID_SD -> unconnected-(U1A-ID_SD-Pad36)
- U1 pad 41: /Compute Module/DC_GPI25 -> unconnected-(U1A-GPIO25-Pad41)
- U1 pad 45: /Compute Module/BL_GPIO24 -> unconnected-(U1A-GPIO24-Pad45)
- U1 pad 48: /Compute Module/RST_GPIO27 -> unconnected-(U1A-GPIO27-Pad48)
- U1 pad 49: /Compute Module/CS_GPIO18 -> unconnected-(U1A-GPIO18-Pad49)
- U1 pad 78: /Compute Module/GPIO_VREF -> +3V3

Commit message: Revised USB design 1xUSB-C 2.0, 2xUSB-A 3.0
Parts:
- removed the C16 at (117.9, 169.5)
- removed C20: 100nF, Screenly:C_0402
- removed the C26 at (127.2, 147.9)
- removed the D3 at (70.1, 141.3)
- removed the D4 at (73.0, 141.3)
- removed the R14 at (127.2, 149.8)
- removed the R15 at (127.2, 151.7)
- added C39: 100nF, Screenly:C_0402, F.Cu at (154.7, 165.5)
- added C40: 10uF, Screenly:C_1210, F.Cu at (170.0, 166.6)
- added C41: 100nF, Screenly:C_0402, F.Cu at (154.7, 167.4)
- added C42: 100nF, Screenly:C_0402, F.Cu at (154.7, 169.4)
- added C43: 10uF, Screenly:C_1210, F.Cu at (170.0, 170.7)
- added C44: 100nF, Screenly:C_0402, F.Cu at (154.7, 171.3)
- added C45: 100nF, Screenly:C_0402, F.Cu at (159.2, 181.0)
- added C51: 100nF, Screenly:C_0402, F.Cu at (154.7, 173.2)
- added C52: 100nF, Screenly:C_0402, F.Cu at (157.7, 165.5)
- added D11: TPD4E05U06DQAR, Screenly:TI_USON-10_2.5x1.0mm_P0.5mm, F.Cu at (143.1, 166.6)
- added D12: TPD4E05U06DQAR, Screenly:TI_USON-10_2.5x1.0mm_P0.5mm, F.Cu at (146.0, 166.6)
- added D13: TPD4E05U06DQAR, Screenly:TI_USON-10_2.5x1.0mm_P0.5mm, F.Cu at (148.8, 166.6)
- added D14: TPD4E05U06DQAR, Screenly:TI_USON-10_2.5x1.0mm_P0.5mm, F.Cu at (151.7, 166.6)
- added D15: TPD4E05U06DQAR, Screenly:TI_USON-10_2.5x1.0mm_P0.5mm, F.Cu at (160.0, 192.6)
- added J10: TYPE-C-31-D-06, Screenly:USB_C_Receptacle_HRO_TYPE-C-31-D-06_Vertical, F.Cu at (170.8, 121.5)
- added J8: USB-A3-S-RA, Screenly:USB_A_USB3_AdamTech_USB-A3-S-RA_Horizontal, F.Cu at (187.5, 124.0)
- added J9: USB-A3-S-RA, Screenly:USB_A_USB3_AdamTech_USB-A3-S-RA_Horizontal, F.Cu at (194.5, 109.5)
- added Q2: 2N7002, Screenly:SOT-23, F.Cu at (156.3, 192.8)
- added R30: 10K, Screenly:R_0402, F.Cu at (157.7, 167.4)
- added R31: 10K, Screenly:R_0402, F.Cu at (157.7, 169.4)
- added R32: 120, Screenly:R_0402, F.Cu at (157.7, 171.3)
- added R33: 120, Screenly:R_0402, F.Cu at (167.3, 177.1)
- added R34: 10K, Screenly:R_0402, F.Cu at (157.7, 173.2)
- added R35: 100K, Screenly:R_0402, F.Cu at (160.8, 165.5)
- added R36: 100K, Screenly:R_0402, F.Cu at (160.8, 167.4)
- added R37: 10K, Screenly:R_0402, F.Cu at (160.8, 169.4)
- added R38: 120, Screenly:R_0402, F.Cu at (160.8, 171.3)
- added R40: 120, Screenly:R_0402, F.Cu at (162.3, 177.1)
- added R41: 5.1K, Screenly:R_0402, F.Cu at (162.3, 179.0)
- added R42: 5.1K, Screenly:R_0402, F.Cu at (162.3, 181.0)
- added R43: 120, Screenly:R_0402, F.Cu at (162.3, 182.9)
- added R44: 5.1K, Screenly:R_0402, F.Cu at (171.5, 144.0)
- added R45: 5.1K, Screenly:R_0402, F.Cu at (171.5, 142.1)
- added R47: 100K, Screenly:R_0402, F.Cu at (162.3, 184.8)
- added U8: AP22653W6-7, Screenly:SOT-23-6, F.Cu at (164.8, 166.8)
- added U9: AP22653W6-7, Screenly:SOT-23-6, F.Cu at (164.8, 171.2)
- J7: value 10.0 QHHTZB6.3 -> HYCW275-USBC24-050B; footprint Screenly:USB_A_SHOUHAN_QHHTZB6.3_Horizontal -> Screenly:USB_C_Receptacle_HOAUC_HYCW275-USBC24-050B
- R28: value 100K -> 31.6K
- U7: value AP22652W6-7 -> AP22653W6-7
- moved U7 39.8 mm to (151.1, 196.9)
- moved R28 38.7 mm to (159.2, 184.8)
- moved R29 38.7 mm to (159.2, 186.7)
- moved R26 38.7 mm to (159.2, 182.9)
- moved C36 37.1 mm to (159.2, 177.1)
- moved C38 37.1 mm to (159.2, 179.0)
- moved C37 33.7 mm to (151.4, 192.6)
- moved C17 8.59 mm to (249.2, 55.1)
- moved C18 8.59 mm to (249.2, 59.2)
- moved C24 8.59 mm to (249.2, 67.4)
- moved C25 8.59 mm to (249.2, 71.4)
- moved C23 8.59 mm to (249.2, 63.3)
- moved R16 8.59 mm to (253.5, 65.6)
- moved C22 8.59 mm to (253.5, 57.9)
- moved C28 8.59 mm to (253.5, 59.8)
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Connections:
- net /USB/~{USBA_PWR_FAULT} renamed /Compute Module/~{USBA_PWR_FAULT}
- C36 pad 1: Net-(J7-VBUS) -> Net-(U7-OUT)
- C37 pad 1: Net-(J7-VBUS) -> Net-(U7-OUT)
- C38 pad 1: +5V -> +5V_USB
- J7 pad SH: unconnected-(J7-PadSH) -> GND
- U1 pad 111: /Compute Module/VBUS_EN -> Net-(U1B-VBUS_EN)
- U7 pad 1: +5V -> +5V_USB
- U7 pad 3: GND -> Net-(Q2-D)
- U7 pad 6: Net-(J7-VBUS) -> Net-(U7-OUT)

Commit message: Finished schematics design.
Parts:
- added C43: 100nF, Screenly:C_0402, F.Cu at (35.1, 77.3)
- added C44: 100nF, Screenly:C_0402, F.Cu at (35.1, 79.3)
- added C49: 100nF, Screenly:C_0402, F.Cu at (64.5, 95.5)
- added C50: 100nF, Screenly:C_0402, F.Cu at (64.5, 97.4)
- added C51: 100nF, Screenly:C_0402, F.Cu at (64.5, 99.3)
- added C52: 1uF, Screenly:C_0402, F.Cu at (64.5, 93.6)
- added C53: 100nF, Screenly:C_0402, F.Cu at (70.0, 49.5)
- added C54: 100nF, Screenly:C_0402, F.Cu at (70.0, 51.4)
- added C55: 10uF, Screenly:C_1210, F.Cu at (54.3, 66.6)
- added C56: 100nF, Screenly:C_0402, F.Cu at (68.6, 83.9)
- added C57: 100nF, Screenly:C_0402, F.Cu at (45.1, 77.3)
- added C58: 10uF, Screenly:C_1210, F.Cu at (49.4, 78.4)
- added C59: 10uF, Screenly:C_1210, F.Cu at (49.4, 90.7)
- added C60: 10uF, Screenly:C_1210, F.Cu at (49.4, 82.5)
- added C61: 10uF, Screenly:C_1210, F.Cu at (49.4, 86.6)
- added C62: 100nF, Screenly:C_0402, F.Cu at (45.1, 81.2)
- added C63: 100nF, Screenly:C_0402, F.Cu at (45.1, 83.1)
- added C64: 2.2uF, Screenly:C_0603, F.Cu at (48.6, 94.0)
- added C65: 2.2uF, Screenly:C_0603, F.Cu at (48.6, 96.5)
- added C66: 100nF, Screenly:C_0402, F.Cu at (45.1, 79.3)
- added C67: 2.2nF, Screenly:C_0402, F.Cu at (45.1, 85.0)
- added C68: 2.2nF, Screenly:C_0402, F.Cu at (45.1, 87.0)
- added D15: Green, Screenly:LED_LiteOn_LTST-S270_SideView, F.Cu at (39.2, 78.0)
- added D16: Red, Screenly:LED_LiteOn_LTST-S270_SideView, F.Cu at (39.2, 81.1)
- added D17: PESD5V0U2BT, Screenly:SOT-23, F.Cu at (38.8, 84.9)
- added J12: 0472192001, Screenly:microSD_HC_Molex_47219-2001, F.Cu at (60.0, 57.1)
- added J13: PJ-320A-4P, Screenly:Jack_3.5mm_SHOUHAN_PJ-320A-4P_Horizontal, F.Cu at (56.1, 79.2)
- added J2: BM03B-SRSS-TB, Screenly:JST_SH_BM03B-SRSS-TB_1x03-1MP_P1.00mm_Vertical, F.Cu at (50.0, 130.1)
- added R12: 10K, Screenly:R_0402, F.Cu at (31.5, 97.2)
- added R2: 33R, Screenly:R_0402, F.Cu at (24.5, 73.4)
- added R3: 120, Screenly:R_0402, F.Cu at (47.6, 134.2)
- added R4: 120, Screenly:R_0402, F.Cu at (47.6, 136.1)
- added R41: 10K, Screenly:R_0402, F.Cu at (35.1, 83.1)
- added R42: 120, Screenly:R_0402, F.Cu at (35.1, 81.2)
- added R43: 1K, Screenly:R_0402, F.Cu at (35.1, 88.9)
- added R5: 33R, Screenly:R_0402, F.Cu at (24.5, 71.5)
- added R54: 56K, Screenly:R_0402, F.Cu at (67.5, 144.7)
- added R55: 56K, Screenly:R_0402, F.Cu at (67.5, 146.6)
- added R56: 10K, Screenly:R_0402, F.Cu at (64.5, 101.3)
- added R57: 10K, Screenly:R_0402, F.Cu at (64.5, 105.1)
- added R58: 10K, Screenly:R_0402, F.Cu at (64.5, 103.2)
- added R59: 120, Screenly:R_0402, F.Cu at (70.0, 53.3)
- added R60: 10K, Screenly:R_0402, F.Cu at (70.0, 55.2)
- added R61: 31.6K, Screenly:R_0402, F.Cu at (70.0, 57.1)
- added R62: 5.1K, Screenly:R_0402, F.Cu at (68.6, 85.8)
- added R63: 5.1K, Screenly:R_0402, F.Cu at (68.6, 87.7)
- added R64: 1K, Screenly:R_0402, F.Cu at (68.6, 89.7)
- added R65: 10K, Screenly:R_0402, F.Cu at (45.1, 92.7)
- added R66: 470, Screenly:R_0402, F.Cu at (45.1, 88.9)
- added R67: 470, Screenly:R_0402, F.Cu at (45.1, 90.8)
- added SW1: PTS645VM31-2, Screenly:SW_Tactile_SPST_Angled_PTS645Vx31-2LFS, F.Cu at (26.0, 80.3)
- added SW2: PTS645VM31-2, Screenly:SW_Tactile_SPST_Angled_PTS645Vx31-2LFS, F.Cu at (26.0, 89.2)
- added TP1: TestPoint, Screenly:TestPoint_Pad_D2.0mm, B.Cu at (31.2, 171.6)
- added TP10: TestPoint, Screenly:TestPoint_Pad_D2.0mm, B.Cu at (37.3, 171.6)
- added TP11: TestPoint, Screenly:TestPoint_Pad_D2.0mm, B.Cu at (37.3, 175.7)
- added TP12: TestPoint, Screenly:TestPoint_Pad_D2.0mm, B.Cu at (37.3, 179.7)
- added TP13: TestPoint, Screenly:TestPoint_Pad_D2.0mm, B.Cu at (41.4, 189.8)
- added TP14: TestPoint, Screenly:TestPoint_Pad_D2.0mm, B.Cu at (41.4, 193.8)
- added TP15: TestPoint, Screenly:TestPoint_Pad_D2.0mm, B.Cu at (35.3, 189.8)
- added TP16: TestPoint, Screenly:TestPoint_Pad_D2.0mm, B.Cu at (35.3, 193.8)
- added TP17: TestPoint, Screenly:TestPoint_Pad_D2.0mm, B.Cu at (47.4, 171.6)
- added TP18: TestPoint, Screenly:TestPoint_Pad_D2.0mm, B.Cu at (47.4, 175.7)
- added TP19: TestPoint, Screenly:TestPoint_Pad_D2.0mm, B.Cu at (47.4, 179.7)
- added TP2: TestPoint, Screenly:TestPoint_Pad_D2.0mm, B.Cu at (31.2, 175.7)
- added TP20: TestPoint, Screenly:TestPoint_Pad_D2.0mm, B.Cu at (47.4, 183.8)
- added TP21: TestPoint, Screenly:TestPoint_Pad_D2.0mm, B.Cu at (56.5, 171.6)
- added TP22: TestPoint, Screenly:TestPoint_Pad_D2.0mm, B.Cu at (56.5, 175.7)
- added TP23: TestPoint, Screenly:TestPoint_Pad_D2.0mm, B.Cu at (56.5, 179.7)
- added TP24: TestPoint, Screenly:TestPoint_Pad_D2.0mm, B.Cu at (56.5, 183.8)
- added TP25: TestPoint, Screenly:TestPoint_Pad_D2.0mm, B.Cu at (56.5, 187.8)
- added TP26: TestPoint, Screenly:TestPoint_Pad_D2.0mm, B.Cu at (56.5, 193.8)
- added TP27: TestPoint, Screenly:TestPoint_Pad_D2.0mm, B.Cu at (21.0, 180.6)
- added TP28: TestPoint, Screenly:TestPoint_Pad_D2.0mm, B.Cu at (21.0, 176.5)
- added TP29: TestPoint, Screenly:TestPoint_Pad_D2.0mm, B.Cu at (47.4, 189.8)
- added TP3: TestPoint, Screenly:TestPoint_Pad_D2.0mm, B.Cu at (26.3, 175.9)
- added TP30: TestPoint, Screenly:TestPoint_Pad_D2.0mm, B.Cu at (21.0, 172.5)
- added TP4: TestPoint, Screenly:TestPoint_Pad_D2.0mm, B.Cu at (26.3, 171.8)
- added TP5: TestPoint, Screenly:TestPoint_Pad_D2.0mm, B.Cu at (31.2, 179.7)
- added TP6: TestPoint, Screenly:TestPoint_Pad_D2.0mm, B.Cu at (41.4, 171.6)
- added TP7: TestPoint, Screenly:TestPoint_Pad_D2.0mm, B.Cu at (41.4, 175.7)
- added TP8: TestPoint, Screenly:TestPoint_Pad_D2.0mm, B.Cu at (41.4, 179.7)
- added TP9: TestPoint, Screenly:TestPoint_Pad_D2.0mm, B.Cu at (41.4, 183.8)
- added U10: SLB9672XU20FW1624, Screenly:Infineon_PG-UQFN-32-1_5x5mm_P0.5mm_EP3.6x3.6mm, F.Cu at (69.6, 96.1)
- added U11: AP22653W6-7, Screenly:SOT-23-6, F.Cu at (59.6, 66.8)
- added U12: M24C64-RMN6TP, Screenly:SOIC-8_3.9x4.9mm_P1.27mm, F.Cu at (73.2, 74.2)
- added U13: PCM5102APWR, Screenly:TSSOP-20_4.4x6.5mm_P0.65mm, F.Cu at (56.6, 96.9)
- J1: value CR2032 Holder -> CR2032 Retainer; footprint Screenly:BatteryHolder_MYOUNG_BS-02_CR2032 -> Screenly:BatteryHolder_MYOUNG_MY-2032-08_CR2032
- R44, R45: value 5.1K -> 1K
- U5, U6: value AP22652W6-7 -> AP22653W6-7
- moved U5 215.1 mm to (25.5, 98.4)
- moved U6 215.1 mm to (25.5, 102.9)
- moved R44 148.6 mm to (35.1, 85.0), turned to 0 degrees
- moved R45 147.1 mm to (35.1, 87.0), turned to 0 degrees
- moved R14 31.3 mm to (58.8, 129.2)
- moved R16 31.3 mm to (58.8, 131.2)
- moved J1 7.00 mm to (185.0, 84.0), turned to 90 degrees
- moved C18 6.34 mm to (66.8, 129.2)
- moved R19 6.34 mm to (66.8, 133.0)
- moved R20 6.34 mm to (66.8, 131.1)
- moved J5 6.03 mm to (176.2, 57.0)
- moved U1 3.76 mm to (121.2, 72.2)
- renumbered C16 to C1, C11 to C10, C5 to C11, C6 to C13, C13 to C14, C7 to C15, C14 to C16, C29 to C17, C27 to C18, C17 to C19, C1 to C2, C18 to C20, C19 to C21, C28 to C22, C21 to C23, C26 to C24, C22 to C25, C23 to C26, C24 to C27, C25 to C28, C30 to C29, C8 to C3, C32 to C30, C34 to C31, C35 to C32, C31 to C33, C33 to C34, C39 to C35, C42 to C36, C51 to C37, C52 to C38, C40 to C39, C2 to C4, C43 to C40, C44 to C42, C38 to C45, C45 to C46, C37 to C47, C36 to C48, C9 to C5, C3 to C6, C10 to C7, C15 to C8, C4 to C9, D13 to D12, D12 to D13, D15 to D18, D8 to D6, D6 to D7, D9 to D8, D7 to D9, J7 to J11, J2 to J3, J3 to J4, J4 to J5, J5 to J6, J6 to J7, R14 to R1, R1 to R10, R3 to R13, R4 to R14, R8 to R15, R9 to R16, R5 to R17, R10 to R18, R18 to R19, R17 to R20, R20 to R21, R19 to R22, R15 to R23, R12 to R24, R13 to R25, R16 to R26, R22 to R27, R23 to R28, R24 to R29, R25 to R30, R21 to R31, R27 to R32, R35 to R33, R36 to R34, R30 to R35, R34 to R36, R31 to R37, R37 to R38, R32 to R39, R38 to R40, R43 to R46, R40 to R48, R29 to R49, R28 to R50, R41 to R51, R42 to R52, R26 to R53, R33 to R6, R6 to R8, R2 to R9, U8 to U7, U9 to U8, U7 to U9
Connections:
- D10 pad 6: /Compute Module/HDMI1.HOTPLUG -> unconnected-(D10-Pad6)
- D10 pad 7: /Compute Module/HDMI1.CEC -> unconnected-(D10-Pad7)
- D11 pad 6: /Compute Module/USB3_0.RX_N -> unconnected-(D11-Pad6)
- D11 pad 7: /Compute Module/USB3_0.RX_P -> unconnected-(D11-Pad7)
- D12 pad 6: /Compute Module/USB3_1.RX_N -> unconnected-(D12-Pad6)
- D12 pad 7: /Compute Module/USB3_1.RX_P -> unconnected-(D12-Pad7)
- D13 pad 4: unconnected-(D12-D2+-Pad4) -> unconnected-(D13-D2+-Pad4)
- D13 pad 5: unconnected-(D12-D2--Pad5) -> unconnected-(D13-D2--Pad5)
- D13 pad 6: unconnected-(D12-D2--Pad5) -> unconnected-(D13-Pad6)
- D13 pad 7: unconnected-(D12-D2+-Pad4) -> unconnected-(D13-Pad7)
- D14 pad 6: unconnected-(D14-D2--Pad5) -> unconnected-(D14-Pad6)
- D14 pad 7: unconnected-(D14-D2+-Pad4) -> unconnected-(D14-Pad7)
- D18 pad 1: /Compute Module/USB2.D_N -> /Compute Module/USB2.D_P
- D18 pad 10: /Compute Module/USB2.D_N -> /Compute Module/USB2.D_P
- D18 pad 2: /Compute Module/USB2.D_P -> /Compute Module/USB2.D_N
- D18 pad 4: unconnected-(D15-D2+-Pad4) -> unconnected-(D18-D2+-Pad4)
- D18 pad 5: unconnected-(D15-D2--Pad5) -> unconnected-(D18-D2--Pad5)
- D18 pad 6: unconnected-(D15-D2--Pad5) -> unconnected-(D18-Pad6)
- D18 pad 7: unconnected-(D15-D2+-Pad4) -> unconnected-(D18-Pad7)
- D18 pad 9: /Compute Module/USB2.D_P -> /Compute Module/USB2.D_N
- D3 pad 6: /Compute Module/ETH.TRD1_N -> unconnected-(D3-Pad6)
- D3 pad 7: /Compute Module/ETH.TRD1_P -> unconnected-(D3-Pad7)
- D4 pad 6: /Compute Module/ETH.TRD3_N -> unconnected-(D4-Pad6)
- D4 pad 7: /Compute Module/ETH.TRD3_P -> unconnected-(D4-Pad7)
- D5 pad 6: /Compute Module/HDMI0.D1_N -> unconnected-(D5-Pad6)
- D5 pad 7: /Compute Module/HDMI0.D1_P -> unconnected-(D5-Pad7)
- D6 pad 6: /Compute Module/HDMI1.D1_N -> unconnected-(D6-Pad6)
- D6 pad 7: /Compute Module/HDMI1.D1_P -> unconnected-(D6-Pad7)
- D7 pad 6: /Compute Module/HDMI0.CK_N -> unconnected-(D7-Pad6)
- D7 pad 7: /Compute Module/HDMI0.CK_P -> unconnected-(D7-Pad7)
- D8 pad 6: /Compute Module/HDMI1.CK_N -> unconnected-(D8-Pad6)
- D8 pad 7: /Compute Module/HDMI1.CK_P -> unconnected-(D8-Pad7)
- D9 pad 6: /Compute Module/HDMI0.HOTPLUG -> unconnected-(D9-Pad6)
- D9 pad 7: /Compute Module/HDMI0.CEC -> unconnected-(D9-Pad7)
- J11 pad A5: Net-(J7-CC1) -> Net-(J11-CC1)
- J11 pad A6: /Compute Module/USB2.D_N -> /Compute Module/USB2.D_P
- J11 pad A7: /Compute Module/USB2.D_P -> /Compute Module/USB2.D_N
- J11 pad B5: Net-(J7-CC2) -> Net-(J11-CC2)
- J11 pad B6: /Compute Module/USB2.D_N -> /Compute Module/USB2.D_P
- J11 pad B7: /Compute Module/USB2.D_P -> /Compute Module/USB2.D_N
- R44 pad 1: GND -> Net-(D15-A)
- R44 pad 2: Net-(J7-CC1) -> +3V3
- R45 pad 1: Net-(J7-CC2) -> Net-(D16-A)
- R45 pad 2: GND -> +3V3
- R49 pad 2: /Compute Module/~{USBA_PWR_FAULT} -> /Compute Module/~{USB2_PWR_FAULT}
- R53 pad 2: /Compute Module/~{USBA_PWR_FAULT} -> /Compute Module/~{USB2_PWR_FAULT}
- U1 pad 100: /Compute Module/CAM_GPIO1 -> unconnected-(U1A-CAM_GPIO1-Pad100)
- U1 pad 101: /Compute Module/USBOTG_ID -> unconnected-(U1B-USB_OTG_ID-Pad101)
- U1 pad 115: /Compute Module/DPHY0_P.D0_N -> unconnected-(U1B-MIPI0_D0_N-Pad115)
- U1 pad 117: /Compute Module/DPHY0_P.D0_P -> unconnected-(U1B-MIPI0_D0_P-Pad117)
- U1 pad 121: /Compute Module/DPHY0_P.D1_N -> unconnected-(U1B-MIPI0_D1_N-Pad121)
- U1 pad 123: /Compute Module/DPHY0_P.D1_P -> unconnected-(U1B-MIPI0_D1_P-Pad123)
- U1 pad 127: /Compute Module/DPHY0_P.C_N -> unconnected-(U1B-MIPI0_C_N-Pad127)
- U1 pad 129: /Compute Module/DPHY0_P.C_P -> unconnected-(U1B-MIPI0_C_P-Pad129)
- U1 pad 133: /Compute Module/DPHY0_P.D2_N -> unconnected-(U1B-MIPI0_D2_N-Pad133)
- U1 pad 135: /Compute Module/DPHY0_P.D2_P -> unconnected-(U1B-MIPI0_D2_P-Pad135)
- U1 pad 139: /Compute Module/DPHY0_P.D3_N -> unconnected-(U1B-MIPI0_D3_N-Pad139)
- U1 pad 141: /Compute Module/DPHY0_P.D3_P -> unconnected-(U1B-MIPI0_D3_P-Pad141)
- U1 pad 175: /Compute Module/DPHY1_P.D0_N -> unconnected-(U1B-MIPI1_D0_N-Pad175)
- U1 pad 177: /Compute Module/DPHY1_P.D0_P -> unconnected-(U1B-MIPI1_D0_P-Pad177)
- U1 pad 181: /Compute Module/DPHY1_P.D1_N -> unconnected-(U1B-MIPI1_D1_N-Pad181)
- U1 pad 183: /Compute Module/DPHY1_P.D1_P -> unconnected-(U1B-MIPI1_D1_P-Pad183)
- U1 pad 187: /Compute Module/DPHY1_P.C_N -> unconnected-(U1B-MIPI1_C_N-Pad187)
- U1 pad 189: /Compute Module/DPHY1_P.C_P -> unconnected-(U1B-MIPI1_C_P-Pad189)
- U1 pad 193: /Compute Module/DPHY1_P.D2_N -> unconnected-(U1B-MIPI1_D2_N-Pad193)
- U1 pad 194: /Compute Module/DPHY1_P.D3_N -> unconnected-(U1B-MIPI1_D3_N-Pad194)
- U1 pad 195: /Compute Module/DPHY1_P.D2_P -> unconnected-(U1B-MIPI1_D2_P-Pad195)
- U1 pad 196: /Compute Module/DPHY1_P.D3_P -> unconnected-(U1B-MIPI1_D3_P-Pad196)
- U1 pad 24: unconnected-(U1A-GPIO26-Pad24) -> /PCIE_PG
- U1 pad 25: /Compute Module/SCLK_GPIO21 -> /Analog Audio/Audio.SDO0
- U1 pad 26: /Compute Module/MISO_GPIO19 -> /Compute Module/A_WS
- U1 pad 27: /Compute Module/MOSI_GPIO20 -> unconnected-(U1A-GPIO20-Pad27)
- U1 pad 30: unconnected-(U1A-GPIO6-Pad30) -> /Compute Module/~{HDMI1_PWR_FAULT}
- U1 pad 34: unconnected-(U1A-GPIO5-Pad34) -> /Compute Module/~{HDMI0_PWR_FAULT}
- U1 pad 35: unconnected-(U1A-ID_SC-Pad35) -> /Compute Module/EE_SCL
- U1 pad 36: unconnected-(U1A-ID_SD-Pad36) -> /Compute Module/EE_SDA
- U1 pad 37: unconnected-(U1A-GPIO7-Pad37) -> /Compute Module/TPM.~{CS}
- U1 pad 38: unconnected-(U1A-GPIO11-Pad38) -> /Compute Module/TPM.CLK
- U1 pad 40: unconnected-(U1A-GPIO9-Pad40) -> /Compute Module/TPM.MISO
- U1 pad 41: unconnected-(U1A-GPIO25-Pad41) -> /Compute Module/~{TPM_PIRQ}
- U1 pad 44: unconnected-(U1A-GPIO10-Pad44) -> /Compute Module/TPM.MOSI
- U1 pad 45: unconnected-(U1A-GPIO24-Pad45) -> /Compute Module/~{TPM_RST}
- U1 pad 46: unconnected-(U1A-GPIO22-Pad46) -> /Compute Module/~{USB3_0_PWR_FAULT}
- U1 pad 47: unconnected-(U1A-GPIO23-Pad47) -> /Compute Module/~{USB3_1_PWR_FAULT}
- U1 pad 48: unconnected-(U1A-GPIO27-Pad48) -> /Compute Module/~{USB2_PWR_FAULT}
- U1 pad 49: unconnected-(U1A-GPIO18-Pad49) -> /Compute Module/A_SCLK
- U1 pad 50: unconnected-(U1A-GPIO17-Pad50) -> /USB_PG
- U1 pad 51: unconnected-(U1A-GPIO15-Pad51) -> /Compute Module/DBG_RX
- U1 pad 54: unconnected-(U1A-GPIO4-Pad54) -> /Compute Module/~{FACTORY_RST_BTN}
- U1 pad 55: unconnected-(U1A-GPIO14-Pad55) -> /Compute Module/DBG_TX
- U1 pad 64: /Compute Module/SD_CARD.D5 -> unconnected-(U1A-SD_DAT5-Pad64)
- U1 pad 68: /Compute Module/SD_CARD.D4 -> unconnected-(U1A-SD_DAT4-Pad68)
- U1 pad 70: /Compute Module/SD_CARD.D7 -> unconnected-(U1A-SD_DAT7-Pad70)
- U1 pad 72: /Compute Module/SD_CARD.D6 -> unconnected-(U1A-SD_DAT6-Pad72)
- U1 pad 94: /Compute Module/CC1 -> unconnected-(U1A-CC1-Pad94)
- U1 pad 96: /Compute Module/CC2 -> unconnected-(U1A-CC2-Pad96)
- U1 pad 99: /Compute Module/GLOBAL_EN -> unconnected-(U1A-PMIC_ENABLE-Pad99)
- U5 pad 3: GND -> +5V
- U6 pad 3: GND -> +5V

Commit message: New square shape
Added Raspberry Pi Antenna Kit
Parts:
- added MK1: Antenna Kit Outline, Screenly:RaspberryPi_Antenna_Kit_Outline_SideView, F.Cu at (82.5, 108.8)
- SW1, SW2: footprint Screenly:SW_Tactile_SPST_Angled_PTS645Vx31-2LFS -> Screenly:SW_Tactile_SPST_Angled_PTS645Vx58-2LFS
- moved SW1 84.3 mm to (87.8, 137.8), turned to 90 degrees
- moved SW2 74.4 mm to (91.8, 54.2), turned to 90 degrees
- moved D16 66.4 mm to (85.8, 128.5), turned to 90 degrees
- moved D15 65.8 mm to (85.8, 124.5), turned to 90 degrees
- moved C49 62.1 mm to (7.10, 119.1)
- moved C50 62.1 mm to (7.10, 121.0)
- moved C51 62.1 mm to (7.10, 122.9)
- moved C52 62.1 mm to (7.10, 117.1)
- moved C53 62.1 mm to (12.6, 73.0)
- moved C55 62.1 mm to (-3.10, 90.2)
- moved C56 62.1 mm to (11.2, 107.5)
- moved C57 62.1 mm to (-12.3, 100.9)
- moved C62 62.1 mm to (-12.3, 104.8)
- moved C63 62.1 mm to (-12.3, 106.7)
- moved C66 62.1 mm to (-12.3, 102.8)
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Other:
- board size 120 x 90 mm -> 120 x 120 mm

Commit message: Rough placements
Parts:
- added J14: DF40HC(3.0)-100DS-0.4V, Screenly:Hirose_DF40HC-3.0-100DS-0.4V_2x50_P0.4mm_Vertical_NoCopper, F.Cu at (122.5, 63.0)
- added J15: DF40HC(3.0)-100DS-0.4V, Screenly:Hirose_DF40HC-3.0-100DS-0.4V_2x50_P0.4mm_Vertical_NoCopper, F.Cu at (122.5, 97.0)
- moved R12 243.7 mm to (217.7, 120.5)
- moved R16 197.8 mm to (208.0, 121.7)
- moved C1 166.7 mm to (83.0, 99.9)
- moved U6 166.7 mm to (131.8, 157.4)
- moved R2 155.6 mm to (120.4, 70.5)
- moved R5 155.6 mm to (120.4, 68.6)
- moved D3 152.5 mm to (94.0, 118.3), turned to 90 degrees
- moved D4 151.9 mm to (97.5, 118.3), turned to 90 degrees
- moved R1 147.3 mm to (126.0, 67.3)
- moved U5 143.9 mm to (109.0, 150.9)
- moved U11 136.5 mm to (114.5, 12.9)
- moved C55 136.5 mm to (109.3, 12.7)
- moved C10 130.6 mm to (214.6, 102.9)
- moved C12 130.6 mm to (214.6, 104.9)
- moved C14 130.6 mm to (195.1, 120.8)
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Connections:
- D1 pad 1: GND -> Net-(D1-A1)
- D1 pad 2: Net-(D1-A2) -> GND
- D10 pad 6: unconnected-(D10-Pad6) -> /Compute Module/HDMI1.HOTPLUG
- D10 pad 7: unconnected-(D10-Pad7) -> /Compute Module/HDMI1.CEC
- D11 pad 6: unconnected-(D11-Pad6) -> /Compute Module/USB3_0.RX_N
- D11 pad 7: unconnected-(D11-Pad7) -> /Compute Module/USB3_0.RX_P
- D12 pad 6: unconnected-(D12-Pad6) -> /Compute Module/USB3_1.RX_N
- D12 pad 7: unconnected-(D12-Pad7) -> /Compute Module/USB3_1.RX_P
- D13 pad 6: unconnected-(D13-Pad6) -> unconnected-(D13-D2--Pad5)
- D13 pad 7: unconnected-(D13-Pad7) -> unconnected-(D13-D2+-Pad4)
- D14 pad 6: unconnected-(D14-Pad6) -> unconnected-(D14-D2--Pad5)
- D14 pad 7: unconnected-(D14-Pad7) -> unconnected-(D14-D2+-Pad4)
- D18 pad 6: unconnected-(D18-Pad6) -> unconnected-(D18-D2--Pad5)
- D18 pad 7: unconnected-(D18-Pad7) -> unconnected-(D18-D2+-Pad4)
- D3 pad 4: /Compute Module/ETH.TRD1_P -> /Compute Module/ETH.TRD1_N
- D3 pad 5: /Compute Module/ETH.TRD1_N -> /Compute Module/ETH.TRD1_P
- D3 pad 6: unconnected-(D3-Pad6) -> /Compute Module/ETH.TRD1_P
- D3 pad 7: unconnected-(D3-Pad7) -> /Compute Module/ETH.TRD1_N
- D4 pad 4: /Compute Module/ETH.TRD3_P -> /Compute Module/ETH.TRD3_N
- D4 pad 5: /Compute Module/ETH.TRD3_N -> /Compute Module/ETH.TRD3_P
- D4 pad 6: unconnected-(D4-Pad6) -> /Compute Module/ETH.TRD3_P
- D4 pad 7: unconnected-(D4-Pad7) -> /Compute Module/ETH.TRD3_N
- D5 pad 6: unconnected-(D5-Pad6) -> /Compute Module/HDMI0.D1_N
- D5 pad 7: unconnected-(D5-Pad7) -> /Compute Module/HDMI0.D1_P
- D6 pad 6: unconnected-(D6-Pad6) -> /Compute Module/HDMI1.D1_N
- D6 pad 7: unconnected-(D6-Pad7) -> /Compute Module/HDMI1.D1_P
- D7 pad 6: unconnected-(D7-Pad6) -> /Compute Module/HDMI0.CK_N
- D7 pad 7: unconnected-(D7-Pad7) -> /Compute Module/HDMI0.CK_P
- D8 pad 6: unconnected-(D8-Pad6) -> /Compute Module/HDMI1.CK_N
- D8 pad 7: unconnected-(D8-Pad7) -> /Compute Module/HDMI1.CK_P
- D9 pad 6: unconnected-(D9-Pad6) -> /Compute Module/HDMI0.HOTPLUG
- D9 pad 7: unconnected-(D9-Pad7) -> /Compute Module/HDMI0.CEC
- J3 pad 1: Net-(D1-A2) -> Net-(D1-A1)
- Q1 pad 2: Net-(D1-A2) -> Net-(D1-A1)
- TP7 pad 1: Net-(D1-A2) -> Net-(D1-A1)
Routing:
- net /Compute Module/ETH.TRD0_P: track 0.00 -> 85.7 mm
- net /Compute Module/ETH.TRD0_N: track 0.00 -> 83.4 mm
- net /Compute Module/ETH.TRD1_P: track 0.00 -> 75.9 mm
- net /Compute Module/ETH.TRD1_N: track 0.00 -> 75.9 mm
- net /Compute Module/ETH.TRD2_N: track 0.00 -> 74.5 mm
- net /Compute Module/ETH.TRD2_P: track 0.00 -> 74.4 mm
- net /Compute Module/ETH.TRD3_P: track 0.00 -> 74.0 mm
- net /Compute Module/ETH.TRD3_N: track 0.00 -> 73.9 mm
Other:
- outline, holes or cut-outs redrawn
- copper layers 2 -> 4
